Commit message: Change moveit configuration to not include the grippers.

File: hironx_moveit_config/models/HiroNX.urdf (robot description, URDF)
Before this commit: robot HiroNX, 24 links, 23 joints
Links:
- removed link LHAND_JOINT0_Link
- removed link LHAND_JOINT1_Link
- removed link LHAND_JOINT2_Link
- removed link LHAND_JOINT3_Link
- removed link RHAND_JOINT0_Link
- removed link RHAND_JOINT1_Link
- removed link RHAND_JOINT2_Link
- removed link RHAND_JOINT3_Link
Joints:
- removed joint LHAND_JOINT0
- removed joint LHAND_JOINT1
- removed joint LHAND_JOINT2
- removed joint LHAND_JOINT3
- removed joint RHAND_JOINT0
- removed joint RHAND_JOINT1
- removed joint RHAND_JOINT2
- removed joint RHAND_JOINT3
